Commit message: Foot + Force torque sensor

File: antmodel_description/urdf/antmodel.xacro (robot description, xacro)
@@ -236,5 +236,5 @@
 <mu2>1</mu2>
   </link>
-<!-- Foot -->
+<!-- Foot  sphere
 <link name="tarsus_${suffix}">
 <collision>
@@ -266,4 +266,28 @@
 <mu2>1</mu2>
 </link>
+-->
+<!-- Foot  flat -->
+<link name="tarsus_${suffix}">
+<collision>
+<origin xyz="${2*tibia_rad} 0 0" rpy="0 ${PI/2} 0"/>
+<geometry>
+	<cylinder length="0.0001" radius="${tibia_rad}"/>
+</geometry>
+</collision>
+<visual>
+<origin xyz="${2*tibia_rad} 0 0" rpy="0 ${PI/2} 0"/>
+<geometry>
+	<cylinder length="0.0001" radius="${tibia_rad}"/>
+      </geometry>
+      <material name="black"/>
+</visual>
+<inertial>
+      <origin  xyz="${2*tibia_rad} 0 0" rpy="0 ${PI/2} 0"/>
+      <mass value="${tibia_mass/5}"/>
+    <cylinder_inertia m="${tibia_mass/5}" r="${tibia_rad}" h="${0.0001}"/>
+</inertial>
+<mu>1</mu>
+<mu2>1</mu2>
+</link>
  <!--
   <link name="tarsus_${suffix}">
@@ -439,4 +463,7 @@
   <gazebo reference="base_${suffix}">
     <material>Gazebo/Black</material>
+  </gazebo>
+ <gazebo reference="tarsus_${suffix}">
+    <material>Gazebo/Orange</material>
   </gazebo>
   <!-- Transmission to ROS -->
